Commit message: finally got a urdf to load into gazebo, the issue was a combination of wrong urdf, running through paser was helpful

File: src/testbot_description/urdf/test.urdf (robot description, URDF)
Before this commit: robot test, 3 links, 2 joints
Links:
- removed link link1
- link link0: geometry collision cylinder length=0.5 radius=1; visual box size=1 1 1
Joints:
- removed joint joint1

Commit message: sucessfully loads urdf into gazebo with 3 links, next step is to connect with ros contorl

File: src/testbot_description/urdf/test.urdf (robot description, URDF)
Before this commit: robot test, 2 links, 1 joints
Links:
- added link link1, mass 0.4; collision box size=0.01 0.01 0.2; visual box size=0.01 0.01 0.2
- added link link2, mass 0.4; collision box size=0.01 0.01 0.15; visual box size=0.01 0.01 0.15
- link link0: mass 1 -> 0.4; geometry collision box size=0.08 0.08 0.08; visual box size=0.08 0.08 0.08
Joints:
- added joint joint1: type revolute, parent link0, child link1, origin xyz=0 0 .08 rpy=0 0 0, axis 1 0 0, limit lower=-1.571 upper=1.571 effort=10 velocity=1.0
- added joint joint2: type revolute, parent link1, child link2, origin xyz=0 0 .2 rpy=0 0 0, axis 1 0 0, limit lower=-1.571 upper=1.571 effort=10 velocity=1.0
